File: AtmegaPCB/AtmegaPCB.kicad_sch (KiCad schematic)
At the start: 14 parts

Commit message: USB Start
Parts:
- added USB?: (no value), symbol Type-C:HRO-TYPE-C-31-M-12
- C?: value (none) -> 1uF
- C?: value (none) -> 22pF
- C? (x2): value (none) -> 0.1uF
- C?: value (none) -> 10uF
- R? (x2): value (none) -> 10k
- R? (x2): value (none) -> 22
- SW?: value (none) -> SW_Push
- U?: value (none) -> ATmega32U4-A; footprint (none) -> Package_QFP:TQFP-44_10x10mm_P0.8mm
- Y?: value (none) -> 16MHz
Connections:
- net D+: now also R?.2, U?.4 (D+); no longer R?.1
- net D-: now also R?.2, U?.3 (D-); no longer R?.1
- new net: R?.1, USB?.5 (DN2), USB?.7 (DN1)
- new net: R?.1, USB?.6 (DP1), USB?.8 (DP2)
- new net: USB?.1 (GND), USB?.12 (GND), USB?.13 (SHIELD)
- new net: USB?.11 (VBUS), USB?.2 (VBUS)
Other:
- moved on the sheet: R?
