File: AtmegaPCB/AtmegaPCB.kicad_sch (KiCad schematic)
At the start: 175 parts, among them SW1 SW_Push, U1 PRTR5V0U2X, U2 ATmega32U4-A, Y1 16MHz

Commit message: Matrix Start
Parts:
- MX65: footprint MX_Alps_Hybrid:MX-1U-NoLED -> (none)
- MX66: footprint MX_Alps_Hybrid:MX-2.75U-NoLED -> (none)
Changed lines of the file:
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@@
       (effects (font (size 0.508 0.508)))
     )
-    (property "Footprint" "MX_Alps_Hybrid:MX-2.75U-NoLED" (id 2) (at 203.2 153.797 0)
+    (property "Footprint" "" (id 2) (at 203.2 153.797 0)
       (effects (font (size 1.524 1.524)) hide)
     )
@@
       (effects (font (size 0.508 0.508)))
     )
-    (property "Footprint" "MX_Alps_Hybrid:MX-1U-NoLED" (id 2) (at 190.373 153.797 0)
+    (property "Footprint" "" (id 2) (at 190.373 153.797 0)
       (effects (font (size 1.524 1.524)) hide)
     )
@@
     )
     (path "/e87c40d9-f420-49a1-8067-ecc2fe34d96e"
-      (reference "MX65") (unit 1) (value "MX-NoLED") (footprint "MX_Alps_Hybrid:MX-1U-NoLED")
+      (reference "MX65") (unit 1) (value "MX-NoLED") (footprint "MX_Alps_Hybrid:MX-2.75U-NoLED")
     )
     (path "/c75dd2cd-8695-4d6a-9129-fb088fec4d8f"
-      (reference "MX66") (unit 1) (value "MX-NoLED") (footprint "MX_Alps_Hybrid:MX-2.75U-NoLED")
+      (reference "MX66") (unit 1) (value "MX-NoLED") (footprint "MX_Alps_Hybrid:MX-1U-NoLED")
     )
     (path "/7e3e0cb4-b1fc-435b-bb48-b266b8669056"

Commit message: Keymap Setup
Parts:
- MX21, MX34: footprint (none) -> MX_Alps_Hybrid:MX-1.5U-NoLED
- MX35: value (none) -> MX-NoLED; footprint (none) -> MX_Alps_Hybrid:MX-1U-NoLED
- MX39: value (none) -> MX-NoLED; footprint (none) -> MX_Alps_Hybrid:MX-1.75U-NoLED
- MX40, MX66: footprint (none) -> MX_Alps_Hybrid:MX-1U-NoLED
- MX51: footprint (none) -> MX_Alps_Hybrid:MX-2.25U-NoLED
- MX65: footprint (none) -> MX_Alps_Hybrid:MX-2.75U-NoLED
Connections:
- net ROW4 is gone; now on net COL17: D67.1 (K), D68.1 (K), D69.1 (K), D70.1 (K), D71.1 (K), D72.1 (K), D73.1 (K), D74.1 (K), D75.1 (K), D76.1 (K), D77.1 (K), D78.1 (K)
- net COL10: no longer MX77.1 (COL)
- net COL11: now also MX73.1 (COL); no longer MX78.1 (COL)
- net COL12: now also MX74.1 (COL)
- net COL13: no longer MX65.1 (COL)
- net COL14: now also MX65.1 (COL), MX75.1 (COL); no longer MX66.1 (COL)
- net COL15: now also MX76.1 (COL)
- net COL16: now also MX17.1 (COL), MX35.1 (COL), MX66.1 (COL), MX77.1 (COL)
- net COL17: now also MX78.1 (COL)
- net COL5: no longer MX72.1 (COL)
- net COL6: no longer MX73.1 (COL)
- net COL7: now also MX72.1 (COL); no longer MX74.1 (COL)
- net COL8: no longer MX75.1 (COL)
- net COL9: no longer MX76.1 (COL)
Other:
- moved on the sheet: C1, C2, C3, C4, C5, C6, C7, D1, D10, D11, D12, D13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

Commit message: Matrix Update2
Parts:
- U1: footprint Package_QFP:TQFP-44_10x10mm_P0.8mm -> (none)
Changed lines of the file:
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@@
   (junction (at 48.895 266.7) (diameter 0) (color 0 0 0 0)
   )
+  (junction (at 53.975 241.3) (diameter 0) (color 0 0 0 0)
+  )
   (junction (at 177.419 168.021) (diameter 0) (color 0 0 0 0)
   )
@@
   (junction (at 292.862 151.511) (diameter 0) (color 0 0 0 0)
   )
+  (junction (at 71.374 241.3) (diameter 0) (color 0 0 0 0)
+  )
   (junction (at 151.765 151.511) (diameter 0) (color 0 0 0 0)
   )
@@
     (stroke (width 0) (type default) (color 0 0 0 0))
   )
-  (wire (pts (xy 51.308 241.3) (xy 57.277 241.3))
+  (wire (pts (xy 51.308 241.3) (xy 53.975 241.3))
     (stroke (width 0) (type default) (color 0 0 0 0))
   )
@@
     (stroke (width 0) (type default) (color 0 0 0 0))
   )
+  (wire (pts (xy 71.374 241.3) (xy 74.93 241.3))
+    (stroke (width 0) (type default) (color 0 0 0 0))
+  )
   (wire (pts (xy 223.901 157.861) (xy 223.901 174.498))
     (stroke (width 0) (type default) (color 0 0 0 0))
@@
     (stroke (width 0) (type default) (color 0 0 0 0))
   )
+  (wire (pts (xy 53.975 241.3) (xy 57.277 241.3))
+    (stroke (width 0) (type default) (color 0 0 0 0))
+  )
   (wire (pts (xy 126.111 151.511) (xy 138.938 151.511))
     (stroke (width 0) (type default) (color 0 0 0 0))
@@
     (stroke (width 0) (type default) (color 0 0 0 0))
   )
-  (wire (pts (xy 68.58 241.3) (xy 74.93 241.3))
+  (wire (pts (xy 68.58 241.3) (xy 71.374 241.3))
     (stroke (width 0) (type default) (color 0 0 0 0))
   )
@@
     (pin "2")
   )
+  (symbol (lib_id "power:PWR_FLAG") (at 71.374 241.3 0) (unit 1)
+    (in_bom yes) (on_board yes)
+    (property "Reference" "#FLG0102" (id 0) (at 71.374 239.395 0)
+      (effects (font (size 1.27 1.27)) hide)
+    )
+    (property "Value" "" (id 1) (at 75.057 237.744 0))
+    (property "Footprint" "" (id 2) (at 71.374 241.3 0)
+      (effects (font (size 1.27 1.27)) hide)
+    )
+    (property "Datasheet" "~" (id 3) (at 71.374 241.3 0)
+      (effects (font (size 1.27 1.27)) hide)
+    )
+    (pin "1")
+  )
   (symbol (lib_id "Device:D_Small") (at 241.554 182.118 90) (unit 1)
     (in_bom yes) (on_board yes)
@@
     (pin "2")
   )
+  (symbol (lib_id "power:PWR_FLAG") (at 53.975 241.3 0) (unit 1)
+    (in_bom yes) (on_board yes)
+    (property "Reference" "#FLG0101" (id 0) (at 53.975 239.395 0)
+      (effects (font (size 1.27 1.27)) hide)
+    )
+    (property "Value" "" (id 1) (at 54.102 233.807 90))
+    (property "Footprint" "" (id 2) (at 53.975 241.3 0)
+      (effects (font (size 1.27 1.27)) hide)
+    )
+    (property "Datasheet" "~" (id 3) (at 53.975 241.3 0)
+      (effects (font (size 1.27 1.27)) hide)
+    )
+    (pin "1")
+  )
   (symbol (lib_id "Device:C_Small") (at 24.003 46.736 90) (unit 1)
     (in_bom yes) (on_board yes)
@@
       (effects (font (size 1.524 1.524)))
     )
-    (property "Footprint" "Package_QFP:TQFP-44_10x10mm_P0.8mm" (id 2) (at 82.042 265.049 0)
+    (property "Footprint" "" (id 2) (at 82.042 265.049 0)
       (effects (font (size 1.524 1.524)) hide)
     )
@@
     (pin "2")
   )
-  (symbol (lib_id "power:+5V") (at 74.93 241.3 0) (unit 1)
-    (in_bom yes) (on_board yes) (fields_autoplaced)
-    (property "Reference" "#PWR04" (id 0) (at 74.93 245.11 0)
+  (symbol (lib_id "power:+5V") (at 74.93 241.3 270) (unit 1)
+    (in_bom yes) (on_board yes)
+    (property "Reference" "#PWR04" (id 0) (at 71.12 241.3 0)
       (effects (font (size 1.27 1.27)) hide)
     )
-    (property "Value" "+5V" (id 1) (at 74.93 237.7242 0))
+    (property "Value" "+5V" (id 1) (at 77.724 241.173 90)
+      (effects (font (size 1.27 1.27)) (justify left))
+    )
     (property "Footprint" "" (id 2) (at 74.93 241.3 0)
       (effects (font (size 1.27 1.27)) hide)
@@
   )
   (symbol_instances
+    (path "/c3bf29a4-6ac8-4b15-a256-a377e3db5183"
+      (reference "#FLG0101") (unit 1) (value "PWR_FLAG") (footprint "")
+    )
+    (path "/b6803b1c-1f0f-4586-adc4-e499dc7c77a4"
+      (reference "#FLG0102") (unit 1) (value "PWR_FLAG") (footprint "")
+    )
     (path "/1c07aaa2-7e68-4a87-a4f4-913d0a552d3a"
       (reference "#PWR01") (unit 1) (value "GND") (footprint "")
@@
     )
     (path "/e699ba9f-e40b-4f88-84c9-f2421fca5f85"
-      (reference "U1") (unit 1) (value "PRTR5V0U2X") (footprint "Package_QFP:TQFP-44_10x10mm_P0.8mm")
+      (reference "U1") (unit 1) (value "PRTR5V0U2X") (footprint "random-keyboard-parts:SOT143B")
     )
     (path "/79504858-1b96-4dd0-9148-59204b6e4598"

Commit message: Traces Started
Parts:
- U1: footprint (none) -> random-keyboard-parts:SOT143B
Connections:
- net COL17: no longer D67.1 (K), D68.1 (K), D69.1 (K), D70.1 (K), D71.1 (K), D72.1 (K), D73.1 (K), D74.1 (K), D75.1 (K), D76.1 (K), D77.1 (K), D78.1 (K)
- net DN: now reaches R2.1, U1.3 (IO2), USB1.5 (DN2), USB1.7 (DN1)
- net DP: now reaches R3.1, U1.2 (IO1), USB1.6 (DP1), USB1.8 (DP2)
- new net ROW4: D67.1 (K), D68.1 (K), D69.1 (K), D70.1 (K), D71.1 (K), D72.1 (K), D73.1 (K), D74.1 (K), D75.1 (K), D76.1 (K), D77.1 (K), D78.1 (K)
Changed lines of the file:
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@@
   (junction (at 318.516 201.168) (diameter 0) (color 0 0 0 0)
   )
-  (junction (at 344.043 201.168) (diameter 0) (color 0 0 0 0)
-  )
   (junction (at 56.261 143.002) (diameter 0) (color 0 0 0 0)
   )
@@
   (junction (at 159.766 174.498) (diameter 0) (color 0 0 0 0)
   )
-  (junction (at 352.044 201.168) (diameter 0) (color 0 0 0 0)
-  )
   (junction (at 211.074 125.095) (diameter 0) (color 0 0 0 0)
   )
@@
   (junction (at 288.036 157.861) (diameter 0) (color 0 0 0 0)
   )
-  (junction (at 352.044 191.008) (diameter 0) (color 0 0 0 0)
-  )
   (junction (at 249.555 157.861) (diameter 0) (color 0 0 0 0)
   )
@@
     (stroke (width 0) (type default) (color 0 0 0 0))
   )
-  (wire (pts (xy 344.043 201.168) (xy 352.044 201.168))
-    (stroke (width 0) (type default) (color 0 0 0 0))
-  )
   (wire (pts (xy 56.261 143.002) (xy 56.261 142.875))
     (stroke (width 0) (type default) (color 0 0 0 0))
@@
     (stroke (width 0) (type default) (color 0 0 0 0))
   )
-  (wire (pts (xy 391.795 201.168) (xy 391.795 203.962))
-    (stroke (width 0) (type default) (color 0 0 0 0))
-  )
   (wire (pts (xy 300.863 117.475) (xy 300.863 125.095))
     (stroke (width 0) (type default) (color 0 0 0 0))
@@
     (stroke (width 0) (type default) (color 0 0 0 0))
   )
-  (wire (pts (xy 352.044 191.008) (xy 352.044 201.168))
-    (stroke (width 0) (type default) (color 0 0 0 0))
-  )
   (wire (pts (xy 164.592 201.168) (xy 177.419 201.168))
     (stroke (width 0) (type default) (color 0 0 0 0))
@@
     (stroke (width 0) (type default) (color 0 0 0 0))
   )
-  (wire (pts (xy 352.044 201.168) (xy 391.795 201.168))
-    (stroke (width 0) (type default) (color 0 0 0 0))
-  )
   (wire (pts (xy 254.381 151.511) (xy 267.208 151.511))
     (stroke (width 0) (type default) (color 0 0 0 0))
@@
     )
   )
+  (global_label "DN" (shape input) (at 65.786 254 90) (fields_autoplaced)
+    (effects (font (size 1.27 1.27)) (justify left))
+    (property "Intersheet References" "${INTERSHEET_REFS}" (id 0) (at 65.7066 248.9864 90)
+      (effects (font (size 1.27 1.27)) (justify left) hide)
+    )
+  )
   (global_label "COL16" (shape input) (at 339.217 117.475 90) (fields_autoplaced)
     (effects (font (size 1.27 1.27)) (justify left))
@@
     )
   )
+  (global_label "DP" (shape input) (at 66.04 256.54 270) (fields_autoplaced)
+    (effects (font (size 1.27 1.27)) (justify right))
+    (property "Intersheet References" "${INTERSHEET_REFS}" (id 0) (at 65.9606 261.4931 90)
+      (effects (font (size 1.27 1.27)) (justify right) hide)
+    )
+  )
   (global_label "ROW4" (shape input) (at 120.269 201.168 180) (fields_autoplaced)
     (effects (font (size 1.27 1.27)) (justify right))
@@
       (effects (font (size 1.27 1.27)) hide)
     )
-    (property "Value" "" (id 1) (at 75.057 237.744 0))
+    (property "Value" "PWR_FLAG" (id 1) (at 75.057 237.744 0))
     (property "Footprint" "" (id 2) (at 71.374 241.3 0)
       (effects (font (size 1.27 1.27)) hide)
@@
       (effects (font (size 1.27 1.27)) hide)
     )
-    (property "Value" "" (id 1) (at 54.102 233.807 90))
+    (property "Value" "PWR_FLAG" (id 1) (at 54.102 233.807 90))
     (property "Footprint" "" (id 2) (at 53.975 241.3 0)
       (effects (font (size 1.27 1.27)) hide)
@@
       (effects (font (size 1.524 1.524)))
     )
-    (property "Footprint" "" (id 2) (at 82.042 265.049 0)
+    (property "Footprint" "random-keyboard-parts:SOT143B" (id 2) (at 82.042 265.049 0)
       (effects (font (size 1.524 1.524)) hide)
     )
