File: AtmegaPCB/AtmegaPCB.kicad_pcb (KiCad board)
At the start: 2 copper layers, 173 parts, among them SW1 SW_Push, U1 PRTR5V0U2X, U2 ATmega32U4-A, Y1 16MHz

Commit message: Matrix Start
Parts:
- added D78: SOD-123, Diode_SMD:D_SOD-123, B.Cu at (413.5, 109.5)
- added MX78: MX-NoLED, MX_Alps_Hybrid:MX-1U-NoLED, F.Cu at (405.6, 109.5)
- D1, D10, D11, D12, D13, D14, D15, D16, D17, D18, D19, D2, D20, D21, D22, D23, D24, D25, D26, D27, D28, D29, D3, D30, D31, D32, D33, D34, D35, D36, D37, D38, D39, D4, D40, D41, D42, D43, D44, D45, D46, D47, D48, D49, D5, D50, D51, D52, D53, D54, D55, D56, D57, D58, D59, D6, D60, D61, D62, D63, D64, D65, D66, D67, D68, D69, D7, D70, D71, D72, D73, D74, D75, D76, D77, D8, D9: moved to B.Cu
- MX21, MX34: footprint MX_Alps_Hybrid:MX-1U-NoLED -> MX_Alps_Hybrid:MX-1.5U-NoLED
- MX38: footprint MX_Alps_Hybrid:MX-1.75U-NoLED -> MX_Alps_Hybrid:MX-1U-NoLED
- MX39: footprint MX_Alps_Hybrid:MX-1U-NoLED -> MX_Alps_Hybrid:MX-1.75U-NoLED
- MX50, MX53: footprint MX_Alps_Hybrid:MX-2.25U-NoLED -> MX_Alps_Hybrid:MX-1U-NoLED
- MX51, MX54: footprint MX_Alps_Hybrid:MX-1U-NoLED -> MX_Alps_Hybrid:MX-2.25U-NoLED
- moved MX65 398.4 mm to (341.3, 90.5)
- moved D77 397.7 mm to (394.5, 109.6), turned to 90 degrees
- moved MX67 395.8 mm to (34.1, 109.5)
- moved D66 393.1 mm to (394.5, 90.5), turned to 90 degrees
- moved D18 358.1 mm to (413.5, 33.3), turned to 90 degrees
- moved MX75 356.3 mm to (331.8, 109.5)
- moved D65 351.6 mm to (349.2, 90.5), turned to 90 degrees
- moved MX35 348.7 mm to (386.6, 52.4)
- moved MX76 345.0 mm to (367.5, 109.5)
- moved D36 344.4 mm to (413.5, 52.4), turned to 90 degrees
- moved D35 342.5 mm to (394.5, 52.4), turned to 90 degrees
- moved D17 339.2 mm to (394.5, 33.3), turned to 90 degrees
- moved D76 338.2 mm to (375.4, 109.5), turned to 90 degrees
- moved MX73 337.5 mm to (284.2, 109.5)
- moved MX64 335.7 mm to (305.6, 90.5)
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Connections:
- D36 pad 1: ROW2 -> ROW1
- D51 pad 1: ROW3 -> ROW2
- MX17 pad 1: COL16 -> unconnected-(MX17-Pad1)
- MX35 pad 1: COL16 -> unconnected-(MX35-Pad1)
- MX36 pad 1: COL0 -> COL17
- MX37 pad 1: COL1 -> COL0
- MX38 pad 1: COL2 -> COL1
- MX39 pad 1: COL3 -> COL2
- MX40 pad 1: COL4 -> COL3
- MX41 pad 1: COL5 -> COL4
- MX42 pad 1: COL6 -> COL5
- MX43 pad 1: COL7 -> COL6
- MX44 pad 1: COL8 -> COL7
- MX45 pad 1: COL9 -> COL8
- MX46 pad 1: COL10 -> COL9
- MX47 pad 1: COL11 -> COL10
- MX48 pad 1: COL12 -> COL11
- MX49 pad 1: COL13 -> COL12
- MX50 pad 1: COL14 -> COL13
- MX51 pad 1: COL0 -> COL14
- MX52 pad 1: COL1 -> COL0
- MX53 pad 1: COL2 -> COL1
- MX54 pad 1: COL3 -> COL2
- MX55 pad 1: COL4 -> COL3
- MX56 pad 1: COL5 -> COL4
- MX57 pad 1: COL6 -> COL5
- MX58 pad 1: COL7 -> COL6
- MX59 pad 1: COL8 -> COL7
- MX60 pad 1: COL9 -> COL8
- MX61 pad 1: COL10 -> COL9
- MX62 pad 1: COL11 -> COL10
- MX63 pad 1: COL12 -> COL11
- MX64 pad 1: COL13 -> COL12
- MX65 pad 1: COL14 -> COL13
- MX66 pad 1: unconnected-(MX66-Pad1) -> COL14

Commit message: Keymap Setup
Parts:
- moved D62 83.7 mm to (331.8, 152.4)
- moved D66 83.7 mm to (450.9, 152.4)
- moved MX62 83.7 mm to (323.9, 152.4)
- moved MX66 83.7 mm to (442.9, 152.4)
- moved D17 83.7 mm to (450.9, 95.2)
- moved MX17 83.7 mm to (442.9, 95.2)
- moved D10 83.7 mm to (288.9, 95.2)
- moved D11 83.7 mm to (308.0, 95.2)
- moved D31 83.7 mm to (355.6, 114.3)
- moved D35 83.7 mm to (450.9, 114.3)
- moved D5 83.7 mm to (193.7, 95.2)
- moved D50 83.7 mm to (379.4, 133.3)
- moved D56 83.7 mm to (217.5, 152.4)
- moved D58 83.7 mm to (255.6, 152.4)
- moved D7 83.7 mm to (231.8, 95.2)
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Connections:
- D67 pad 1: ROW4 -> COL17
- D68 pad 1: ROW4 -> COL17
- D69 pad 1: ROW4 -> COL17
- D70 pad 1: ROW4 -> COL17
- D71 pad 1: ROW4 -> COL17
- D72 pad 1: ROW4 -> COL17
- D73 pad 1: ROW4 -> COL17
- D74 pad 1: ROW4 -> COL17
- D75 pad 1: ROW4 -> COL17
- D76 pad 1: ROW4 -> COL17
- D77 pad 1: ROW4 -> COL17
- D78 pad 1: ROW4 -> COL17
- MX17 pad 1: unconnected-(MX17-Pad1) -> COL16
- MX35 pad 1: unconnected-(MX35-Pad1) -> COL16
- MX65 pad 1: COL13 -> COL14
- MX66 pad 1: COL14 -> COL16
- MX72 pad 1: COL5 -> COL7
- MX73 pad 1: COL6 -> COL11
- MX74 pad 1: COL7 -> COL12
- MX75 pad 1: COL8 -> COL14
- MX76 pad 1: COL9 -> COL15
- MX77 pad 1: COL10 -> COL16
- MX78 pad 1: COL11 -> COL17

Commit message: Matrix Update2
Parts:
- F1, R4, R5, U2, USB1, Y1: moved to B.Cu
- U1: footprint Package_QFP:TQFP-44_10x10mm_P0.8mm -> random-keyboard-parts:SOT143B; moved to B.Cu
- moved C1 308.7 mm to (348.2, 232.1)
- moved C2 308.7 mm to (289.3, 235.2)
- moved C3 308.7 mm to (339.7, 240.5)
- moved C4 308.7 mm to (300.9, 225.1)
- moved C5 308.7 mm to (293.9, 231.8)
- moved C6 308.7 mm to (295.2, 228.5)
- moved C7 308.7 mm to (289.4, 231.8)
- moved R1 308.7 mm to (299.6, 228.4)
- moved R2 308.7 mm to (342.9, 246.9)
- moved R3 308.7 mm to (272.6, 228.1)
- moved R6 308.7 mm to (324.4, 204.2)
- moved SW1 294.8 mm to (234.4, 229.3), turned to 90 degrees
- moved U2 286.3 mm to (299.3, 171.3), turned to -90 degrees
- moved Y1 250.5 mm to (259.6, 200.5), turned to 90 degrees
- moved U1 240.7 mm to (290.5, 99.2), turned to 180 degrees
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
Commit message: Routed Vertical Traces
Parts:
- C1, C2, C3, C4, C5, C6, C7, R1, R2, R3, R6, SW1: moved to B.Cu
- moved R2 100.4 mm to (288.3, 162.6), turned to -90 degrees
- moved SW1 98.4 mm to (310.9, 167.4), turned to -90 degrees
- moved C3 89.6 mm to (293.9, 163.5), turned to 180 degrees
- moved C1 71.5 mm to (303.6, 176.2)
- moved C2 69.1 mm to (303.4, 167.5), turned to 180 degrees
- moved R3 68.0 mm to (290.7, 162.6), turned to -90 degrees
- moved C7 67.9 mm to (282.0, 164.3)
- moved R1 64.9 mm to (299.9, 163.5), turned to 180 degrees
- moved C6 62.4 mm to (282.0, 167.5)
- moved C5 62.3 mm to (282.0, 170.7)
- moved C4 54.7 mm to (282.0, 173.8)
- moved Y1 52.5 mm to (303.9, 172.3), turned to 0 degrees
- moved R6 49.6 mm to (282.0, 178.5), turned to 90 degrees
- moved D1 9.53 mm to (108.0, 95.2)
- moved D19 9.53 mm to (108.0, 114.3)
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Routing:
- net COL14: track 0.00 -> 94.2 mm
- net COL3: track 0.00 -> 88.7 mm
- net COL15: track 0.00 -> 86.4 mm
- net COL4: track 0.00 -> 86.2 mm
- net COL7: track 0.00 -> 83.4 mm
- net COL12: track 0.00 -> 83.4 mm
- net COL11: track 0.00 -> 82.3 mm
- net COL2: track 0.00 -> 80.3 mm
- net COL17: track 0.00 -> 74.4 mm
- net COL16: track 0.00 -> 73.4 mm
- net COL1: track 0.00 -> 72.5 mm
- net COL0: track 0.00 -> 72.5 mm
- net COL9: track 0.00 -> 64.3 mm
- net COL6: track 0.00 -> 64.3 mm
- net COL5: track 0.00 -> 64.3 mm
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Other:
- board outline added: 381 x 99.2 mm

Commit message: Traces Started
Parts:
- moved C7 23.1 mm to (300.0, 178.8), turned to 90 degrees
- moved C4 22.2 mm to (303.2, 167.3), turned to -90 degrees
- moved D72 16.0 mm to (261.1, 169.8)
- moved SW1 14.3 mm to (325.2, 166.8)
- moved C1 7.83 mm to (308.1, 169.9), turned to 180 degrees
- moved C2 7.30 mm to (308.1, 173.0)
- moved C5 4.71 mm to (281.0, 175.3), turned to 90 degrees
- moved C6 3.78 mm to (284.0, 164.3), turned to 180 degrees
- moved R2 3.17 mm to (288.3, 159.4)
- moved R3 3.17 mm to (290.7, 159.4)
- moved R5 1.82 mm to (286.4, 92.9)
- moved R6 1.41 mm to (283.4, 178.5)
- moved C3 1.13 mm to (292.7, 163.5)
- moved R1 1.03 mm to (300.9, 163.5)
- moved F1 0.88 mm to (285.8, 100.2), turned to -90 degrees
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Connections:
- net Net-(R2-Pad1) renamed DN
- net Net-(R3-Pad1) renamed DP
- D67 pad 1: COL17 -> ROW4
- D68 pad 1: COL17 -> ROW4
- D69 pad 1: COL17 -> ROW4
- D70 pad 1: COL17 -> ROW4
- D71 pad 1: COL17 -> ROW4
- D72 pad 1: COL17 -> ROW4
- D73 pad 1: COL17 -> ROW4
- D74 pad 1: COL17 -> ROW4
- D75 pad 1: COL17 -> ROW4
- D76 pad 1: COL17 -> ROW4
- D77 pad 1: COL17 -> ROW4
- D78 pad 1: COL17 -> ROW4
Routing:
- net ROW1: track 0.00 -> 373.7 mm, vias 0 -> 2
- net ROW0: track 0.00 -> 373.5 mm, vias 0 -> 2
- net ROW3: track 0.00 -> 354.5 mm, vias 0 -> 3
- net ROW2: track 0.00 -> 310.7 mm, vias 0 -> 2
- net ROW4: track 0.00 -> 280.6 mm
- net GND: track 0.00 -> 215.6 mm, vias 0 -> 4
- net COL0: track 72.5 -> 257.0 mm, vias 0 -> 1
- net +5V: track 0.00 -> 168.2 mm, vias 0 -> 5
- net COL1: track 72.5 -> 240.7 mm, vias 0 -> 1
- net COL17: track 74.4 -> 238.2 mm, vias 0 -> 1
- net COL16: track 73.4 -> 219.2 mm, vias 0 -> 1
- net COL2: track 80.3 -> 216.6 mm, vias 0 -> 1
- net COL15: track 86.4 -> 212.6 mm, vias 0 -> 1
- net COL13: track 42.2 -> 162.9 mm, vias 0 -> 1
- net COL3: track 88.7 -> 201.6 mm, vias 0 -> 1
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- added copper zone on B.Cu, net GND

Commit message: COL & ROW Traced
Parts:
- moved C7 3.13 mm to (298.4, 176.1)
- moved C1 3.09 mm to (308.1, 166.8)
- moved C2 3.09 mm to (308.1, 169.9)
- moved C6 3.09 mm to (284.0, 161.2)
- moved R6 3.09 mm to (283.4, 175.4)
- moved U2 3.09 mm to (292.0, 169.1)
- moved Y1 3.09 mm to (303.6, 168.8)
- moved C3 3.09 mm to (292.7, 160.4)
- moved C4 3.09 mm to (303.2, 164.2)
- moved C5 3.09 mm to (281.0, 172.2)
- moved R1 3.09 mm to (300.9, 160.4)
- moved R2 1.26 mm to (287.3, 158.6)
- moved R3 1.26 mm to (289.7, 158.6)
Connections:
- U2 pad 10: unconnected-(U2-Pad10) -> ROW2
- U2 pad 11: unconnected-(U2-Pad11) -> ROW1
- U2 pad 12: unconnected-(U2-Pad12) -> ROW0
- U2 pad 18: unconnected-(U2-Pad18) -> COL9
- U2 pad 19: unconnected-(U2-Pad19) -> COL10
- U2 pad 20: unconnected-(U2-Pad20) -> COL11
- U2 pad 21: unconnected-(U2-Pad21) -> COL12
- U2 pad 22: unconnected-(U2-Pad22) -> COL13
- U2 pad 25: unconnected-(U2-Pad25) -> COL14
- U2 pad 26: unconnected-(U2-Pad26) -> COL15
- U2 pad 27: unconnected-(U2-Pad27) -> COL16
- U2 pad 28: unconnected-(U2-Pad28) -> COL17
- U2 pad 29: unconnected-(U2-Pad29) -> COL0
- U2 pad 30: unconnected-(U2-Pad30) -> COL1
- U2 pad 31: unconnected-(U2-Pad31) -> COL2
- U2 pad 32: unconnected-(U2-Pad32) -> COL3
- U2 pad 36: unconnected-(U2-Pad36) -> COL4
- U2 pad 37: unconnected-(U2-Pad37) -> COL5
- U2 pad 38: unconnected-(U2-Pad38) -> COL6
- U2 pad 39: unconnected-(U2-Pad39) -> COL7
- U2 pad 40: unconnected-(U2-Pad40) -> ROW4
- U2 pad 41: unconnected-(U2-Pad41) -> ROW3
Routing:
- net ROW4: track 280.6 -> 409.8 mm, vias 0 -> 2
- net ROW0: track 373.5 -> 458.8 mm, vias 2 -> 6
- net ROW1: track 373.7 -> 429.5 mm, vias 2 -> 5
- net ROW2: track 310.7 -> 344.4 mm
- net COL0: track 257.0 -> 282.3 mm
- net COL1: track 240.7 -> 263.7 mm
- net COL2: track 216.6 -> 237.2 mm
- net COL4: track 174.9 -> 194.5 mm
- net ROW3: track 354.5 -> 373.4 mm
- net COL3: track 201.6 -> 220.3 mm
- net COL5: track 138.4 -> 156.8 mm
- net COL17: track 238.2 -> 255.8 mm
- net COL16: track 219.2 -> 236.5 mm
- net COL6: track 119.3 -> 136.6 mm
- net COL15: track 212.6 -> 229.6 mm
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
Commit message: Traces Completed
Parts:
- moved SW1 3.22 mm to (325.7, 169.9)
Routing:
- net Net-(R1-Pad2): track 7.02 -> 32.5 mm, vias 0 -> 2
- net GND: track 211.0 -> 233.3 mm
- net +5V: track 171.0 -> 178.9 mm
Changed lines of the file:
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@@
   )
   (footprint "random-keyboard-parts:SKQG-1155865" (layer "B.Cu")
-    (at 325.175 166.7625 -90)
+    (at 325.7 169.9375 -90)
     (property "Sheetfile" "AtmegaPCB.kicad_sch")
     (property "Sheetname" "")
@@
   (via (at 292.89375 102.39375) (size 0.8) (drill 0.4) (layers "F.Cu" "B.Cu") (net 1))
   (segment (start 298.45 175.10625) (end 296.29375 175.10625) (width 0.381) (layer "B.Cu") (net 1))
+  (segment (start 327.55 173.0375) (end 327.55 174.1) (width 0.381) (layer "B.Cu") (net 1))
   (segment (start 291.19375 165.86875) (end 295.051228 165.86875) (width 0.381) (layer "B.Cu") (net 1))
   (segment (start 291.15625 165.83125) (end 291.19375 165.86875) (width 0.381) (layer "B.Cu") (net 1))
@@
   (segment (start 288.13125 171.5375) (end 287.4 172.26875) (width 0.381) (layer "B.Cu") (net 1))
   (segment (start 304.48125 169.63125) (end 304.48125 169.95) (width 0.381) (layer "B.Cu") (net 1))
+  (segment (start 327.55 174.1) (end 326.23125 175.41875) (width 0.381) (layer "B.Cu") (net 1))
   (segment (start 291.7875 160.425) (end 291.15625 161.05625) (width 0.381) (layer "B.Cu") (net 1))
   (segment (start 286.1925 82.9375) (end 286.1925 87.1175) (width 0.381) (layer "B.Cu") (net 1))
+  (segment (start 312.03125 169.95) (end 309.08125 169.95) (width 0.381) (layer "B.Cu") (net 1))
   (segment (start 291.15625 168.5125) (end 288.13125 171.5375) (width 0.381) (layer "B.Cu") (net 1))
   (segment (start 295.95625 174.76875) (end 295.95625 173.3125) (width 0.381) (layer "B.Cu") (net 1))
@@
   (segment (start 291.15625 165.83125) (end 291.15625 168.5125) (width 0.381) (layer "B.Cu") (net 1))
   (segment (start 302.78125 167.93125) (end 304.48125 169.63125) (width 0.381) (layer "B.Cu") (net 1))
+  (segment (start 317.5 175.41875) (end 312.03125 169.95) (width 0.381) (layer "B.Cu") (net 1))
   (segment (start 309.08125 169.95) (end 307.96623 168.83498) (width 0.381) (layer "B.Cu") (net 1))
   (segment (start 285.5125 90.725) (end 285.5125 92.86875) (width 0.381) (layer "B.Cu") (net 1))
@@
   (segment (start 283.36875 160.90625) (end 283.05625 161.21875) (width 0.381) (layer "B.Cu") (net 1))
   (segment (start 287.4 172.26875) (end 286.25625 172.26875) (width 0.381) (layer "B.Cu") (net 1))
+  (segment (start 326.23125 175.41875) (end 317.5 175.41875) (width 0.381) (layer "B.Cu") (net 1))
   (segment (start 295.95625 173.3125) (end 291.15625 168.5125) (width 0.381) (layer "B.Cu") (net 1))
   (segment (start 286.3725 87.1175) (end 287.2875 88.0325) (width 0.381) (layer "B.Cu") (net 1))
@@
   (segment (start 291.95625 163.36875) (end 291.95625 162.15625) (width 0.25) (layer "B.Cu") (net 4))
   (segment (start 279.4 159.63125) (end 279.4 173.125) (width 0.381) (layer "F.Cu") (net 5))
-  (segment (start 304.00625 159.63125) (end 304.00625 174.7125) (width 0.381) (layer "F.Cu") (net 5))
+  (segment (start 302.41875 176.3) (end 300.74375 176.3) (width 0.381) (layer "F.Cu") (net 5))
+  (segment (start 279.4 158.04375) (end 279.4 159.63125) (width 0.381) (layer "F.Cu") (net 5))
+  (segment (start 311.15 167.56875) (end 302.41875 176.3) (width 0.381) (layer "F.Cu") (net 5))
   (segment (start 300.74375 176.3) (end 300.0375 177.00625) (width 0.381) (layer "F.Cu") (net 5))
-  (segment (start 279.4 158.04375) (end 279.4 159.63125) (width 0.381) (layer "F.Cu") (net 5))
-  (segment (start 304.00625 174.7125) (end 302.41875 176.3) (width 0.381) (layer "F.Cu") (net 5))
+  (segment (start 307.26875 159.63125) (end 311.15 163.5125) (width 0.381) (layer "F.Cu") (net 5))
+  (segment (start 304.00625 159.63125) (end 307.26875 159.63125) (width 0.381) (layer "F.Cu") (net 5))
   (segment (start 295.1875 159.63125) (end 304.00625 159.63125) (width 0.381) (layer "F.Cu") (net 5))
+  (segment (start 311.15 163.5125) (end 311.15 167.56875) (width 0.381) (layer "F.Cu") (net 5))
   (segment (start 279.4 159.63125) (end 284.95625 159.63125) (width 0.381) (layer "F.Cu") (net 5))
-  (segment (start 302.41875 176.3) (end 300.74375 176.3) (width 0.381) (layer "F.Cu") (net 5))
   (segment (start 284.95625 159.63125) (end 295.1875 159.63125) (width 0.381) (layer "F.Cu") (net 5))
   (via (at 295.1875 159.63125) (size 0.8) (drill 0.4) (layers "F.Cu" "B.Cu") (net 5))
@@
   (segment (start 464.4625 166.95) (end 467.3125 169.8) (width 0.25) (layer "B.Cu") (net 104))
   (segment (start 467.3125 169.8) (end 469.9 169.8) (width 0.25) (layer "B.Cu") (net 104))
+  (segment (start 307.975 162.71875) (end 300.0375 162.71875) (width 0.25) (layer "F.Cu") (net 105))
+  (via (at 300.0375 162.71875) (size 0.8) (drill 0.4) (layers "F.Cu" "B.Cu") (net 105))
+  (via (at 307.975 162.71875) (size 0.8) (drill 0.4) (layers "F.Cu" "B.Cu") (net 105))
   (segment (start 300.0375 160.425) (end 300.0375 164.4875) (width 0.25) (layer "B.Cu") (net 105))
   (segment (start 298.65625 165.86875) (end 297.65625 165.86875) (width 0.25) (layer "B.Cu") (net 105))
+  (segment (start 312.09375 166.8375) (end 307.975 162.71875) (width 0.25) (layer "B.Cu") (net 105))
   (segment (start 300.0375 164.4875) (end 298.65625 165.86875) (width 0.25) (layer "B.Cu") (net 105))
+  (segment (start 323.85 166.8375) (end 312.09375 166.8375) (width 0.25) (layer "B.Cu") (net 105))
   (segment (start 289.55625 163.36875) (end 289.55625 161.7625) (width 0.2) (layer "B.Cu") (net 106))
   (segment (start 289.55625 161.7625) (end 287.3375 159.54375) (width 0.2) (layer "B.Cu") (net 106))

Commit message: For Review
Routing:
- added copper zone on F.Cu, net GND
Changed lines of the file:
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@@
       (rotate (xyz 0 0 0))
+    )
+    (model "/Users/macuser2/Documents/GitHub/Picies/WirelessPCBProject/marbastlib/3d/Switch_SKQG.step"
+      (offset (xyz 0 0 0))
+      (scale (xyz 1 1 1))
+      (rotate (xyz -90 0 0))
     )
   )
@@
   (segment (start 287.95625 175.68125) (end 287.95625 174.76875) (width 0.25) (layer "B.Cu") (net 121))
   (segment (start 287.3375 176.3) (end 287.95625 175.68125) (width 0.25) (layer "B.Cu") (net 121))
+  (zone (net 1) (net_name "GND") (layer "F.Cu") (hatch edge 0.508)
+    (connect_pads (clearance 0.508))
+    (min_thickness 0.254)
+    (fill (thermal_gap 0.508) (thermal_bridge_width 0.508))
+    (polygon
+      (pts
+        (xy 311.94375 175.50625)
+        (xy 299.24375 175.50625)
+        (xy 299.24375 162.0125)
+        (xy 311.94375 162.0125)
+      )
+    )
+  )
   (zone (net 1) (net_name "GND") (layer "B.Cu") (hatch edge 0.508)
     (connect_pads (clearance 0.508))
@@
       )
     )
+  )
+  (zone (net 1) (net_name "GND") (layer "B.Cu") (hatch edge 0.508)
+    (connect_pads (clearance 0.508))
+    (min_thickness 0.254)
+    (fill (thermal_gap 0.508) (thermal_bridge_width 0.508))
+    (polygon
+      (pts
+        (xy 296.06875 88.9)
+        (xy 284.95625 88.9)
+        (xy 284.95625 81.75625)
+        (xy 296.06875 81.75625)
+      )
+    )
